Commit message: WORKING TELEOP

File: dev_ws/src/my_package/description/gazebo_control.xacro (robot description, xacro)
@@ -9,5 +9,5 @@
             <max_wheel_torque>200</max_wheel_torque>
             <max_wheel_acceleration>10.0</max_wheel_acceleration>
-            <topic>cmd_vel</topic>
+            <topic>/cmd_vel</topic>
             <odom_topic>odom</odom_topic>
             <tf_topic>tf</tf_topic>
@@ -15,4 +15,9 @@
             <child_frame_id>base</child_frame_id>
         </plugin>
+        <plugin name="gz::sim::systems::JointStatePublisher" filename="gz-sim-joint-state-publisher-system">
+            <topic>joint_states</topic>
+            <joint_name>left_wheel_joint</joint_name>
+            <joint_name>right_wheel_joint</joint_name>
+        </plugin>
     </gazebo>
 </robot>

File: dev_ws/src/my_package/description/robot_core.xacro (robot description, xacro)
@@ -15,4 +15,8 @@
     </material>
     <link name="base">
+        <inertial>
+            <mass value="0.1"/>
+            <inertia ixx="0.001" ixy="0" ixz="0" iyy="0.001" iyz="0" izz="0.001"/>
+        </inertial>
     </link>
     <joint name="chasis_joint" type="fixed">
@@ -60,6 +64,6 @@
                 <friction>
                     <ode>
-                        <mu>0</mu>
-                        <mu2>0</mu2>
+                        <mu>1.0</mu>
+                        <mu2>1.0</mu2>
                     </ode>
                 </friction>
@@ -90,6 +94,6 @@
                 <friction>
                     <ode>
-                        <mu>0</mu>
-                        <mu2>0</mu2>
+                        <mu>1.0</mu>
+                        <mu2>1.0</mu2>
                     </ode>
                 </friction>
