Commit message: Working project

File: dev_ws/src/my_package/description/robot_core.xacro (robot description, xacro)
@@ -23,4 +23,10 @@
         </inertial>
     </link>
+    <joint name="base_footprint_joint" type="fixed">
+        <parent link="base"/>
+        <child link="base_footprint"/>
+        <origin xyz="0 0 0" rpy="0 0 0"/>
+    </joint>
+    <link name="base_footprint"></link>
     <joint name="chasis_joint" type="fixed">
         <parent link="base"/>
